File: PCB/ESP8266Wol.kicad_pcb (KiCad board)
At the start: 2 copper layers, 24.6 x 41.8 mm, 26 parts, among them J2 Conn_01x02, J3 Conn_01x02, J4 Conn_01x02, J5 Conn_02x05_Odd_Even, SW1 SW_Push, U1 ESP-12F, U2 AMS1117, U3 PC817, U4 PC817, U5 PC817

Commit message: update silkscreen
Other:
- board text added: "+"
- board text added: "5V"
- board text added: "PWR"
- board text added: "RST"
